File: hardware/detector/implant_detector.kicad_sch (KiCad schematic)
At the start: 65 parts, among them J1 USB-C, J2 Qwiic, J3 SWD (TC2030), J4 SMA, SW1 CAL, SW2 BOOT, U1 FDC2214, U2 FDC2214, U3 STM32F042F6P6, U4 AP2112K-3.3, U5 USBLC6-2SC6, Y1 40MHz

Commit message: Add routed 4-layer detector PCB, fab outputs and renders
Single board: 8-electrode capacitive head (2x FDC2214), STM32F042 with USB-C
power + ROM DFU programming, near-field RF loop at the tip with edge SMA.
Electrodes shrunk to 14x14 mm to open a via channel; head tanks and escapes
are pre-routed deterministically, rest autorouted with Freerouting 1.9.

DRC: 0 errors, 0 unconnected, schematic parity OK. ERC: 0 violations.
Concept / untested, see README.

Co-Authored-By: Claude Opus 5.5 <noreply@anthropic.com>
Parts:
- E1, E2, E3, E4, E5, E6, E7, E8: footprint lid:Electrode_15x15mm -> lid:Electrode_14x14mm
Connections:
- net SNS2: now also U1.15 (IN3A); no longer U1.11 (IN1A)
- net SNS2B: now also U1.16 (IN3B); no longer U1.12 (IN1B)
- net SNS4: now also U2.15 (IN3A); no longer U2.11 (IN1A)
- net SNS4B: now also U2.16 (IN3B); no longer U2.12 (IN1B)
- net SNS5: now also U1.11 (IN1A); no longer U1.13 (IN2A)
- net SNS5B: now also U1.12 (IN1B); no longer U1.14 (IN2B)
- net SNS6: now also U1.13 (IN2A); no longer U1.15 (IN3A)
- net SNS6B: now also U1.14 (IN2B); no longer U1.16 (IN3B)
- net SNS7: now also U2.11 (IN1A); no longer U2.13 (IN2A)
- net SNS7B: now also U2.12 (IN1B); no longer U2.14 (IN2B)
- net SNS8: now also U2.13 (IN2A); no longer U2.15 (IN3A)
- net SNS8B: now also U2.14 (IN2B); no longer U2.16 (IN3B)
Other:
- moved on the sheet: C2, C4, C5, C6, C7, C8, E2, E4, E5, E6, E7, E8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
