File: hardware/fixtures/tem_plate/tem_plate.kicad_pcb (KiCad board)
At the start: 2 copper layers, 100 x 100 mm, 4 parts

Commit message: First fixture session: TEM cell sees the implant at every placement
TEM cell (h = 20 mm): the implanted Nano X shows a ~1 dB, ~40 MHz wide
notch at 1171 MHz at every placement and both orientations (sim: -1.2 dB
at 1185 MHz). Six of seven genuine placements stay within 0.2 dB; one
genuine re-check showed a similar notch near 1230 MHz, cause unknown.
Slot line: a small (-0.13..-0.20 dB) dip at 817-861 MHz at 0 deg only.

Also:
- gen_fixtures.py: TEM landing marks now place the ramp tip where the
  rigid ramp's tab actually lands, with the ramp overlapping the septum by
  4 mm; regenerated TEM boards and assembly step 3.
- nanovna_capture.py: zeros mean "outside the active calibration's span"
  (e.g. slot 1 recalled at power-on); say to `recall 0`.

Co-Authored-By: Claude Opus 5.5 <noreply@anthropic.com>
Other:
- board text added: "ramps overlap the bare strips from below"
- board text removed: "join the ramps along the bare edges"
